File: tactile_schematic/_autosave-tactile_schematic.kicad_sch (KiCad schematic)
At the start: 37 parts, among them IC1 CY8C4145PVI-PS431, J1 Conn_01x02, J2 Conn_01x04, J3 Conn_01x04, J4 Conn_01x02

Commit message: PCB first draft
Parts:
- CE1, CE2, CE3, CE4: footprint PCB Coils:COIL_GENERATOR -> PCB Coils:COIL_GENERATOR_1
- H1, H2, H3, H4, H5, H6, H7, H8: footprint ECE445L:MountingHole_4_40 -> MountingHole:MountingHole_3.2mm_M3_Pad
Changed lines of the file:
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@@
 			)
 		)
-		(property "Footprint" "PCB Coils:COIL_GENERATOR"
+		(property "Footprint" "PCB Coils:COIL_GENERATOR_1"
 			(at 39.0652 107.95 0)
 			(effects
@@
 			)
 		)
-		(property "Footprint" "ECE445L:MountingHole_4_40"
+		(property "Footprint" "MountingHole:MountingHole_3.2mm_M3_Pad"
 			(at 161.29 68.58 0)
 			(effects
@@
 			)
 		)
-		(property "Footprint" "ECE445L:MountingHole_4_40"
+		(property "Footprint" "MountingHole:MountingHole_3.2mm_M3_Pad"
 			(at 175.26 53.34 0)
 			(effects
@@
 			)
 		)
-		(property "Footprint" "ECE445L:MountingHole_4_40"
+		(property "Footprint" "MountingHole:MountingHole_3.2mm_M3_Pad"
 			(at 161.29 76.2 0)
 			(effects
@@
 			)
 		)
-		(property "Footprint" "ECE445L:MountingHole_4_40"
+		(property "Footprint" "MountingHole:MountingHole_3.2mm_M3_Pad"
 			(at 175.26 68.58 0)
 			(effects
@@
 			)
 		)
-		(property "Footprint" "ECE445L:MountingHole_4_40"
+		(property "Footprint" "MountingHole:MountingHole_3.2mm_M3_Pad"
 			(at 175.26 76.2 0)
 			(effects
@@
 			)
 		)
-		(property "Footprint" "PCB Coils:COIL_GENERATOR"
+		(property "Footprint" "PCB Coils:COIL_GENERATOR_1"
 			(at 121.6152 106.68 0)
 			(effects
@@
 			)
 		)
-		(property "Footprint" "ECE445L:MountingHole_4_40"
+		(property "Footprint" "MountingHole:MountingHole_3.2mm_M3_Pad"
 			(at 161.29 60.96 0)
 			(effects
@@
 			)
 		)
-		(property "Footprint" "ECE445L:MountingHole_4_40"
+		(property "Footprint" "MountingHole:MountingHole_3.2mm_M3_Pad"
 			(at 175.26 60.96 0)
 			(effects
@@
 			)
 		)
-		(property "Footprint" "ECE445L:MountingHole_4_40"
+		(property "Footprint" "MountingHole:MountingHole_3.2mm_M3_Pad"
 			(at 161.29 53.34 0)
 			(effects
@@
 			)
 		)
-		(property "Footprint" "PCB Coils:COIL_GENERATOR"
+		(property "Footprint" "PCB Coils:COIL_GENERATOR_1"
 			(at 96.2152 106.68 0)
 			(effects
@@
 			)
 		)
-		(property "Footprint" "PCB Coils:COIL_GENERATOR"
+		(property "Footprint" "PCB Coils:COIL_GENERATOR_1"
 			(at 67.0052 106.68 0)
 			(effects
