File: 0p7W_0p1S_LARGER/tactile_schematic.kicad_pcb (KiCad board)
At the start: 2 copper layers, 145.2 x 85.6 mm, 55 parts, among them IC1 CY8C4145PVI-PS431, J1 Conn_01x03, J2 Conn_01x04, J3 Conn_01x04, J4 Conn_01x03, J5 Conn_ARM_SWD_TagConnect_TC203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

Commit message: make spacing fixes (first two boards)
Parts:
- moved J4 3.24 mm to (196.7, 112.7)
Routing:
- net SHIELD: track 26.8 -> 23.2 mm
- net Net-(J1-Pin_2): track 98.5 -> 95.6 mm
- net Net-(J1-Pin_3): track 69.6 -> 66.9 mm
Other:
- outline, holes or cut-outs redrawn
