File: 0p4W_0p2S_SAME_SIZE/tactile_schematic.kicad_pcb (KiCad board)
At the start: 2 copper layers, 109.6 x 67.4 mm, 55 parts, among them IC1 CY8C4145PVI-PS431, J1 Conn_01x03, J2 Conn_01x04, J3 Conn_01x04, J4 Conn_01x03, J5 Conn_ARM_SWD_TagConnect_TC203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

Commit message: fixed silkscreen
Connections:
- net SHEILD renamed SHIELD
Changed lines of the file:
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@@
 	(net 39 "SCL")
 	(net 40 "SDA")
-	(net 41 "SHEILD")
+	(net 41 "SHIELD")
 	(net 42 "Net-(J1-Pin_2)")
 	(net 43 "unconnected-(IC1-P2.1-Pad11)")
@@
 			(layers "*.Cu" "*.Mask")
 			(remove_unused_layers no)
-			(net 41 "SHEILD")
+			(net 41 "SHIELD")
 			(pinfunction "Pin_1")
 			(pintype "passive")
@@
 			(layers "*.Cu" "*.Mask")
 			(remove_unused_layers no)
-			(net 41 "SHEILD")
+			(net 41 "SHIELD")
 			(pinfunction "Pin_1")
 			(pintype "passive")
@@
 			(size 0.45 1.775)
 			(layers "F.Cu" "F.Mask" "F.Paste")
-			(net 41 "SHEILD")
+			(net 41 "SHIELD")
 			(pinfunction "P2.0")
 			(pintype "passive")
@@
 			(size 0.45 1.775)
 			(layers "F.Cu" "F.Mask" "F.Paste")
-			(net 41 "SHEILD")
+			(net 41 "SHIELD")
 			(pinfunction "P2.7/VREF")
 			(pintype "passive")
@@
 	(zone
 		(net 41)
-		(net_name "SHEILD")
+		(net_name "SHIELD")
 		(layer "F.Cu")
 		(hatch edge 0.5)
@@
 	(zone
 		(net 41)
-		(net_name "SHEILD")
+		(net_name "SHIELD")
 		(layer "B.Cu")
 		(hatch edge 0.5)

Commit message: make spacing fixes (first two boards)
Parts:
- moved J4 4.21 mm to (251.7, 69.8)
Routing:
- net Net-(J1-Pin_2): track 68.8 -> 65.9 mm
- net Net-(J1-Pin_3): track 58.5 -> 56.4 mm
Other:
- outline, holes or cut-outs redrawn
Changed lines of the file:
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@@
 			(psa4output no)
 			(plot_black_and_white yes)
-			(plotinvisibletext no)
 			(sketchpadsonfab no)
 			(plotpadnumbers no)
@@
 	(footprint "Connector_PinHeader_2.00mm:PinHeader_1x03_P2.00mm_Vertical"
 		(layer "F.Cu")
-		(at 252.000001 74 -90)
+		(at 251.7 69.8 -90)
 		(descr "Through hole straight pin header, 1x03, 2.00mm pitch, single row")
 		(tags "Through hole pin header THT 1x03 2.00mm single row")
@@
 	)
 	(gr_line
-		(start 253.389046 70.797682)
-		(end 253.389046 76.284083)
+		(start 247.3 73.100001)
+		(end 247.281698 77.182719)
 		(stroke
 			(width 0.008)
@@
 	(gr_arc
 		(start 264.371724 56.123035)
-		(mid 260.459134 64.641913)
-		(end 253.389046 70.797682)
+		(mid 258.32079 67.110315)
+		(end 247.3 73.1)
 		(stroke
 			(width 0.008)
-			(type default)
+			(type solid)
 		)
 		(layer "Edge.Cuts")
@@
 		(layer "Edge.Cuts")
 	)
-	(gr_line
-		(start 247.281699 77.182719)
-		(end 247.419095 76.284083)
-		(stroke
-			(width 0.008)
-			(type default)
-		)
-		(layer "Edge.Cuts")
-	)
 	(gr_arc
 		(start 206.871633 41.943283)
@@
 		(layer "Edge.Cuts")
 	)
-	(gr_line
-		(start 253.389046 76.284083)
-		(end 247.419095 76.284083)
-		(stroke
-			(width 0.008)
-			(type default)
-		)
-		(layer "Edge.Cuts")
-	)
 	(gr_arc
 		(start 167.872095 63.348564)
@@
 		(start 187.109285 83.390715)
 		(end 187.109285 83.109285)
-		(width 0.2)
+		(width 0.4)
 		(layer "B.Cu")
 		(net 2)
@@
 		(start 187.109285 83.109285)
 		(end 186 82)
-		(width 0.2)
+		(width 0.4)
 		(layer "B.Cu")
 		(net 2)
@@
 		(start 186 82)
 		(end 186 81)
-		(width 0.2)
+		(width 0.4)
 		(layer "B.Cu")
 		(net 2)
@@
 		(start 187.484285 83.765715)
 		(end 187.109285 83.390715)
-		(width 0.2)
+		(width 0.4)
 		(layer "B.Cu")
 		(net 2)
@@
 	(segment
 		(start 241.78072 69.042)
-		(end 242.04436 69.30564)
+		(end 242.53872 69.8)
 		(width 0.2)
 		(layer "F.Cu")
@@
 	)
 	(segment
-		(start 246.73872 74)
-		(end 248.000001 74)
-		(width 0.2)
-		(layer "F.Cu")
-		(net 21)
-	)
-	(segment
 		(start 243.33572 40.126)
 		(end 243.33572 32.101057)
@@
 	)
 	(segment
+		(start 242.53872 69.8)
+		(end 247.7 69.8)
+		(width 0.2)
+		(layer "F.Cu")
+		(net 21)
+	)
+	(segment
 		(start 232.13072 49.976)
 		(end 231.714 49.976)
@@
 	)
 	(segment
-		(start 242.04436 69.30564)
-		(end 246.73872 74)
-		(width 0.2)
-		(layer "F.Cu")
-		(net 21)
-	)
-	(segment
 		(start 243.35546 31.75)
 		(end 238.4 31.75)
@@
 	)
 	(segment
-		(start 249 73)
-		(end 250 74)
-		(width 0.2)
-		(layer "F.Cu")
-		(net 42)
-	)
-	(segment
-		(start 245.925 72.075)
-		(end 246.85 73)
-		(width 0.2)
-		(layer "F.Cu")
-		(net 42)
-	)
-	(segment
 		(start 242.165 50.845)
 		(end 243.167 51.847)
@@
 	)
 	(segment
-		(start 246.425 72.575)
-		(end 245.925 72.075)
+		(start 242.35 68.5)
+		(end 242.674 68.824)
 		(width 0.2)
 		(layer "F.Cu")
@@
 	)
 	(segment
+		(start 248.723999 68.824)
+		(end 249.699999 69.8)
+		(width 0.2)
+		(layer "F.Cu")
+		(net 42)
+	)
+	(segment
 		(start 241.18072 58.382)
 		(end 241.18072 51.82928)
@@
 	)
 	(segment
-		(start 246.51 72.66)
-		(end 246.425 72.575)
-		(width 0.2)
-		(layer "F.Cu")
-		(net 42)
-	)
-	(segment
 		(start 241.18072 51.82928)
 		(end 242.165 50.845)
@@
 	)
 	(segment
-		(start 245.925 72.075)
-		(end 242.35 68.5)
-		(width 0.2)
-		(layer "F.Cu")
-		(net 42)
-	)
-	(segment
 		(start 243.93572 42.831)
 		(end 243.93572 49.07428)
@@
 	)
 	(segment
-		(start 246.85 73)
-		(end 249 73)
+		(start 242.674 68.824)
+		(end 248.723999 68.824)
 		(width 0.2)
 		(layer "F.Cu")
@@
 			"971252e6-017b-4d72-8c99-0e7f02153bab" "98e006b7-7e3c-4442-8ddd-dd9fd7ad492a"
 			"9d7b98f9-6d9c-4b5e-85c5-b31e207fe83b" "a85f860d-5794-419c-8288-e20bba6a0cbf"
-			"ae3ff10d-ec8f-4ccf-b616-e743631008ce" "bd8f1ab8-3f81-4f70-955e-9be0ce075c08"
-			"bea91297-8c29-410e-bcbb-3f0447c0e07a" "c2ca4671-0470-40fe-ad55-c385d0d0ed0f"
-			"c4dbdc97-61d3-4676-938f-ca783d0d2f11" "cf00cf5e-8d0d-4e1b-bbd8-11e2fd325de9"
-			"d39f5704-4995-4953-9a4a-2095d637747c" "d8721b2c-35eb-4aa2-ba8e-2344026d6e65"
-			"de0e7e35-b16c-4273-b9ee-ac981555411a" "df489cbf-11d1-4ea1-9b0a-485b4ab8da24"
+			"ae3ff10d-ec8f-4ccf-b616-e743631008ce" "bea91297-8c29-410e-bcbb-3f0447c0e07a"
+			"c2ca4671-0470-40fe-ad55-c385d0d0ed0f" "c4dbdc97-61d3-4676-938f-ca783d0d2f11"
+			"cf00cf5e-8d0d-4e1b-bbd8-11e2fd325de9" "d39f5704-4995-4953-9a4a-2095d637747c"
+			"d8721b2c-35eb-4aa2-ba8e-2344026d6e65" "df489cbf-11d1-4ea1-9b0a-485b4ab8da24"
 			"dfc1dc29-b257-4686-a35d-cfe998325a2d" "e9406cb6-0d08-4116-96a3-2f74e7a74107"
 			"fa55d47d-d47a-43b8-a36f-71b8ea532bbd" "fc8f53c2-e1a6-4885-89fd-87701cb4a697"

Commit message: more spacing fixes
Routing:
- net SHIELD: track 32.6 -> 27.7 mm
Changed lines of the file:
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@@
-	)
-	(segment
-		(start 182.685505 79.75)
-		(end 183.773005 79.75)
-		(width 0.2)
-		(layer "F.Cu")
-		(net 41)
 	)
 	(segment
@@
 		(width 0.2)
 		(layer "F.Cu")
-		(net 41)
-	)
-	(segment
-		(start 183.773005 79.75)
-		(end 183.874005 79.851)
-		(width 0.2)
-		(layer "F.Cu")
-		(net 41)
-	)
-	(segment
-		(start 183.773005 82.35)
-		(end 182.685505 82.35)
-		(width 0.2)
-		(layer "F.Cu")
-		(net 41)
-	)
-	(segment
-		(start 183.874005 82.249)
-		(end 183.773005 82.35)
-		(width 0.2)
-		(layer "F.Cu")
-		(net 41)
-	)
-	(segment
-		(start 183.874005 79.851)
-		(end 183.874005 82.249)
-		(width 0.2)
-		(layer "F.Cu")
